File: TempReader_w_I2C.kicad_sch/TempReader_w_I2C_Ltuned.kicad_sch.kicad_pcb (KiCad board)
At the start: 4 copper layers, 40 x 47 mm, 42 parts, among them J1 NRF Pin Header, J2 BME Pin Header, U5 MIC5205-3.3YM5, Y1 16MH

Commit message: Trying to send BME data with battery power
Parts:
- removed C12: 1pF, Capacitor_SMD:C_0402_1005Metric_Pad0.74x0.62mm_HandSolder
- removed H2: MountingHole, MountingHole:MountingHole_2.2mm_M2
- added REF**: MountingHole_2.2mm_M2, MountingHole:MountingHole_2.2mm_M2, F.Cu at (158.0, 73.0)
- C10, C11, C5, C6: footprint Capacitor_SMD:C_0402_1005Metric_Pad0.74x0.62mm_HandSolder -> Capacitor_SMD:C_0603_1608Metric_Pad1.08x0.95mm_HandSolder
- L1, L2, L3: footprint Inductor_SMD:L_0402_1005Metric_Pad0.77x0.64mm_HandSolder -> Inductor_SMD:L_0603_1608Metric_Pad1.05x0.95mm_HandSolder
- moved H3 34.3 mm to (192.2, 113.2)
- moved H4 33.8 mm to (158.2, 113.2)
- moved C14 2.75 mm to (167.2, 98.9)
- moved C15 2.72 mm to (167.2, 100.9)
- moved C10 2.71 mm to (177.2, 107.0)
- moved C6 2.01 mm to (183.3, 109.4)
- moved R2 2.00 mm to (170.3, 100.1)
- moved C5 1.56 mm to (182.4, 107.0)
- moved C11 1.28 mm to (178.7, 107.0)
- moved L3 1.22 mm to (183.3, 104.5), turned to 0 degrees
- moved L2 0.78 mm to (179.7, 104.5)
- moved L1 0.46 mm to (181.4, 103.0)
Routing:
- net GND1: track 54.7 -> 45.7 mm, vias 17 -> 11
- net Net-(NRF24L01+1-VDD_PA): track 5.38 -> 0.00 mm
- net PowerIn: track 4.70 -> 0.00 mm
- net Net-(NRF24L01+1-XC1): track 9.46 -> 12.6 mm
- net Net-(NRF24L01+1-XC2): track 9.74 -> 12.5 mm
- net 50 O out: track 33.8 -> 31.1 mm
- net Net-(NRF24L01+1-ANT1): track 2.60 -> 0.00 mm
- net Net-(NRF24L01+1-ANT2): track 2.04 -> 0.00 mm
- net CS_NRF: track 44.2 -> 42.7 mm
- net SPI_MOSI: track 39.1 -> 37.7 mm
- net Net-(C5-Pad1): track 1.17 -> 0.00 mm
- net +3V3: track 57.4 -> 57.1 mm, vias 14 -> 13
Other:
- board size 40 x 47 mm -> 40 x 50 mm
